File: fu740_pcie_gen3.sch (KiCad schematic (older format))
At the start: 1 part, among them U1 FU740-C000

Commit message: Schematic capture update.
Schematic capture update (PCIe Page.)
Parts:
- added C? (x6): 4.7uF, symbol Device:C_Small
- added C? (x4): 10uF, symbol Device:C_Small
- added C? (x16): 0.22uF, symbol Device:C
- added FB? (x2): 120R, symbol Device:Ferrite_Bead
- added FB?: Ferrite_Bead, symbol Device:Ferrite_Bead
- added R? (x2): 0R001, symbol Device:R
- added TP? (x3): TestPoint, symbol Connector:TestPoint
Connections:
- net labels added: GND, VDD_0V9, VDD_1V8, VDD_PCIEVP, VDD_PCIEVPH, VDD_PCIEVPH_N, VDD_PCIEVPH_P, VDD_PCIEVP_N, VDD_PCIEVP_P
- wire segments 0 -> 175
Other:
- note added: "FU740 - PCIe Gen3"
- moved on the sheet: U1F

Commit message: Schematic capture update
Schematic capture update (PCIe)
Parts:
- removed FB?: Ferrite_Bead, symbol Device:Ferrite_Bead
- added C? (x20): 0.1uF, symbol Device:C_Small
Connections:
- net labels added: PCIeUS_RX0_N, PCIeUS_RX0_P, PCIeUS_RX1_N, PCIeUS_RX1_P, PCIeUS_RX2_N, PCIeUS_RX2_P, PCIeUS_RX3_N, PCIeUS_RX3_P, PCIeUS_RX4_N, PCIeUS_RX4_P, PCIeUS_RX5_N, PCIeUS_RX5_P, PCIeUS_RX6_N, PCIeUS_RX6_P, PCIeUS_RX7_N, PCIeUS_RX7_P, PCIeUS_TX0_N, PCIeUS_TX0_P, PCIeUS_TX1_N, PCIeUS_TX1_P, PCIeUS_TX2_N, PCIeUS_TX2_P, PCIeUS_TX3_N, PCIeUS_TX3_P, PCIeUS_TX4_N, PCIeUS_TX4_P, PCIeUS_TX5_N, PCIeUS_TX5_P, PCIeUS_TX6_N, PCIeUS_TX6_P, PCIeUS_TX7_N, PCIeUS_TX7_P, PCIe_0_CLKREQN, PCIe_0_PERSTN, PCIe_0_WAKEN, PCIe_REFCLK_N, PCIe_REFCLK_P, PCIe_TX0_N, PCIe_TX0_P, PCIe_TX1_N, PCIe_TX1_P, PCIe_TX2_N, PCIe_TX2_P, PCIe_TX3_N, PCIe_TX3_P, PCIe_TX4_N, PCIe_TX4_P, PCIe_TX5_N, PCIe_TX5_P, PCIe_TX6_N, PCIe_TX6_P, PCIe_TX7_N, PCIe_TX7_P
- wire segments 175 -> 255

Commit message: Schematic update
Schematic update
Parts:
- added R?: 200R, symbol Device:R
Connections:
- wire segments 255 -> 258
Changed lines of the file:
@@
 	1    0    0    -1
 $EndComp
+$Comp
+L Device:R R?
+U 1 1 61C57EC9
+P 10100 11400
+AR Path="/6145B860/61C57EC9" Ref="R?"  Part="1"
+AR Path="/614B9C8F/61C57EC9" Ref="R?"  Part="1"
+F 0 "R?" H 10300 11450 50  0000 C CNN
+F 1 "200R" H 10300 11350 50  0000 C CNN
+F 2 "" V 10030 11400 50  0001 C CNN
+F 3 "~" H 10100 11400 50  0001 C CNN
+	1    10100 11400
+	1    0    0    -1
+$EndComp
+Wire Wire Line
+	10550 10900 10100 10900
+Wire Wire Line
+	10100 10900 10100 11250
+$Comp
+L power:GND #PWR?
+U 1 1 61CAD96F
+P 10100 11850
+AR Path="/6145B860/61CAD96F" Ref="#PWR?"  Part="1"
+AR Path="/614B9C8F/61CAD96F" Ref="#PWR?"  Part="1"
+F 0 "#PWR?" H 10100 11600 50  0001 C CNN
+F 1 "GND" H 10105 11677 50  0000 C CNN
+F 2 "" H 10100 11850 50  0001 C CNN
+F 3 "" H 10100 11850 50  0001 C CNN
+	1    10100 11850
+	1    0    0    -1
+$EndComp
+Wire Wire Line
+	10100 11550 10100 11850
 $EndSCHEMATC
