File: fu740_misc.sch (KiCad schematic (older format))
At the start: 1 part, among them U1 FU740-C000

Commit message: Schematic capture progress
Schematic capture progress update.
Parts:
- added R?: 0R20, symbol Device:R
- added R?: 100K, symbol Device:R
- added R? (x4): DNP, symbol Device:R
- added R?: 0R, symbol Device:R
Connections:
- net labels added: EN_VDD_SD, GPIO0, GPIO1, GPIO10, GPIO11, GPIO12, GPIO13, GPIO2, GPIO3, GPIO4, GPIO5, GPIO6, GPIO7, GPIO8, GPIO9, JTAG_TCK, JTAG_TDI, JTAG_TDO, JTAG_TMS, PWM0_0, PWM0_1, PWM0_2, PWM0_3, PWM1_0, SD_CD, VDD_1V8
- wire segments 0 -> 105

Commit message: Schematic work progress update
Schematic work progress update
Parts:
- removed R? (x4): DNP, symbol Device:R
- added R? (x4): DNP, symbol Device:R
- added RN? (x3): 33R, symbol Device:R_Pack04
Connections:
- net labels added: I2C0_SCL, I2C0_SDA, I2C1_SCL, I2C1_SDA, PWM1_2, PWM1_3, QSPI0_CS, QSPI0_DQ0, QSPI0_DQ1, QSPI0_DQ2, QSPI0_DQ3, QSPI0_SCK, QSPI1_CS0, QSPI1_CS0_R, QSPI1_CS1, QSPI1_CS1_R, QSPI1_DQ0, QSPI1_DQ0_R, QSPI1_DQ1, QSPI1_DQ1_R, QSPI1_DQ2, QSPI1_DQ2_R, QSPI1_DQ3, QSPI1_DQ3_R, QSPI1_SCK, QSPI1_SCK_R, SPI0_CS0, SPI0_CS0_R, SPI0_DQ0, SPI0_DQ0_R, SPI0_DQ1, SPI0_DQ1_R, SPI0_SCK, SPI0_SCK_R
- wire segments 105 -> 148
- no-connect marks 0 -> 2
